File: multianem16/cta.kicad_pcb (KiCad board)
At the start: 2 copper layers, 268 x 157.5 mm, 243 parts, among them Q1 TIP41, Q10 TIP41, Q11 TIP41, Q12 TIP41, Q13 TIP41, Q14 TIP41, Q15 TIP41, Q16 TIP41, Q2 TIP41, Q3 TIP41, Q4 TIP41, Q5 TIP41, Q6 TIP41, Q7 TIP41, Q8 TIP41, Q9 TIP41, U1 LM324, U10 LM324, U11 LM324, U12 LM324, U13 LM324, U14 LM324, U15 LM324, U16 LM324, U2 LM324, U3 LM324, U4 LM324, U5 LM324, U6 LM324, U7 LM324, U8 LM324, U9 LM324

Commit message: Working on making the multinanem16 board use symmetric power input.
This way I can use more types of op-amps.
Parts:
- Cua1, Cua2, Cua3, Cua4, Cua5: value 10u -> 100n; footprint Capacitor_THT:CP_Radial_D5.0mm_P2.50mm -> Capacitor_THT:C_Rect_L7.2mm_W3.5mm_P5.00mm_FKS2_FKP2_MKS2_MKP2
- JVIN1: value Conn_01x02 -> Conn_01x06; footprint TerminalBlock:TerminalBlock_bornier-2_P5.08mm -> TerminalBlock:TerminalBlock_bornier-6_P5.08mm
- moved Cua5 167.3 mm to (9.88, -21.6), turned to 0 degrees
- moved Cua4 145.9 mm to (1.13, -16.5), turned to 0 degrees
- moved Cua3 123.7 mm to (1.13, -21.6), turned to 0 degrees
- moved Cua2 104.2 mm to (-7.62, -16.5), turned to 0 degrees
- moved Cua1 19.4 mm to (54.6, 61.0), turned to 90 degrees
- moved JVIN1 8.03 mm to (16.5, 81.3)
- moved Rda1 4.58 mm to (58.4, 54.6)
- turned Rdb1 to 270 degrees
Connections:
- Cua1 pad 1: VCC -> VEE
- Cua2 pad 1: VCC -> VEE
- Cua3 pad 1: VCC -> VEE
- Cua4 pad 1: VCC -> VEE
- Cua5 pad 1: VCC -> VEE
- JVIN1 pad 1: GND -> VCC
- U1 pad 11: GND -> VEE
- U2 pad 11: GND -> VEE
- U3 pad 11: GND -> VEE
- U4 pad 11: GND -> VEE
- U5 pad 11: GND -> VEE
Routing:
- net VEE: track 0.00 -> 113.4 mm, vias 0 -> 2
- net GND: track 2510.4 -> 2423.9 mm
- net Net-(Rda1-Pad1): track 6.35 -> 13.8 mm
- net VCC: track 1489.2 -> 1482.1 mm, vias 33 -> 32
- net Net-(Rda1-Pad2): track 7.62 -> 10.2 mm
- removed copper zone on B.Cu, net GND

Commit message: Working on adding symmetric power to the multianem16 board.
Almost done.
Parts:
- removed Cua11: 10u, Capacitor_THT:CP_Radial_D5.0mm_P2.50mm
- removed the Cua12 at (147.3, 130.8)
- added Cub12: 100n, Capacitor_THT:C_Rect_L7.2mm_W3.5mm_P5.00mm_FKS2_FKP2_MKS2_MKP2, F.Cu at (147.2, 257.8)
- added Cub17: 100n, Capacitor_THT:C_Rect_L7.2mm_W3.5mm_P5.00mm_FKS2_FKP2_MKS2_MKP2, F.Cu at (155.9, 252.7)
- Cua10, Cua13, Cua14, Cua15, Cua16, Cua6, Cua7, Cua8, Cua9: value 10u -> 100n; footprint Capacitor_THT:CP_Radial_D5.0mm_P2.50mm -> Capacitor_THT:C_Rect_L7.2mm_W3.5mm_P5.00mm_FKS2_FKP2_MKS2_MKP2
- moved Cua5 186.0 mm to (176.5, 61.0), turned to 90 degrees
- moved Cua4 164.3 mm to (146.1, 61.0), turned to 90 degrees
- moved Cua16 162.8 mm to (155.9, 247.7)
- moved Cua15 152.5 mm to (147.2, 252.7)
- moved Cua14 144.9 mm to (138.4, 257.8)
- moved Cua3 141.1 mm to (115.6, 61.0), turned to 90 degrees
- moved Cua2 120.8 mm to (85.1, 61.0), turned to 90 degrees
- moved Cua13 120.8 mm to (147.2, 247.7)
- moved Cua9 71.1 mm to (-15.2, 129.5), turned to 270 degrees
- moved Rda9 63.5 mm to (-26.7, 132.1)
- moved Rdb9 55.9 mm to (-22.9, 118.1), turned to 90 degrees
- moved Cua8 19.4 mm to (268.0, 61.0), turned to 90 degrees
- moved Cua7 19.4 mm to (237.5, 61.0), turned to 90 degrees
- moved Cua10 19.4 mm to (67.3, 127.0), turned to 270 degrees
- moved Cua6 19.4 mm to (207.0, 61.0), turned to 90 degrees
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- renumbered Cub12 to Cua12
Connections:
- Cua10 pad 1: VCC -> VEE
- Cua12 pad 1: VCC -> VEE
- Cua13 pad 1: VCC -> VEE
- Cua14 pad 1: VCC -> VEE
- Cua15 pad 1: VCC -> VEE
- Cua16 pad 1: VCC -> VEE
- Cua6 pad 1: VCC -> VEE
- Cua7 pad 1: VCC -> VEE
- Cua8 pad 1: VCC -> VEE
- Cua9 pad 1: VCC -> VEE
- JVIN1 pad 3: GND -> VEE
- JVIN1 pad 4: GND -> VEE
- JVIN1 pad 5: VEE -> GND
- JVIN1 pad 6: VEE -> GND
- U10 pad 11: GND -> VEE
- U11 pad 11: GND -> VEE
- U12 pad 11: GND -> VEE
- U13 pad 11: GND -> VEE
- U14 pad 11: GND -> VEE
- U15 pad 11: GND -> VEE
- U16 pad 11: GND -> VEE
- U6 pad 11: GND -> VEE
- U7 pad 11: GND -> VEE
- U8 pad 11: GND -> VEE
- U9 pad 11: GND -> VEE
Routing:
- net VEE: track 113.4 -> 649.4 mm, vias 2 -> 20
- net GND: track 2423.9 -> 2515.1 mm
- net /VO14: track 189.3 -> 166.9 mm
- net VCC: track 1482.1 -> 1498.7 mm
- net Net-(Rda9-Pad1): track 6.35 -> 15.0 mm
- net Net-(Rda10-Pad1): track 6.35 -> 13.8 mm
- net Net-(Rda6-Pad1): track 6.35 -> 13.8 mm
- net Net-(Rda5-Pad1): track 6.35 -> 13.8 mm
- net Net-(Rda3-Pad1): track 6.35 -> 13.8 mm
- net Net-(Rda2-Pad1): track 6.35 -> 13.8 mm
- net Net-(Rda7-Pad1): track 6.35 -> 13.8 mm
- net Net-(Rda4-Pad1): track 6.35 -> 13.8 mm
- net /VO9: track 39.9 -> 32.5 mm
- net Net-(Rda8-Pad1): track 6.35 -> 13.8 mm
- net /VO10: track 69.6 -> 62.9 mm
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
Commit message: Finnished adding Vee to the 16 anemometers board.
Parts:
- added REF**: MountingHole_3mm_Pad, MountingHole:MountingHole_3mm_Pad, F.Cu at (275.6, 20.3)
- added REF**: MountingHole_3mm_Pad, MountingHole:MountingHole_3mm_Pad, F.Cu at (275.6, 167.6)
- added REF**: MountingHole_3mm_Pad, MountingHole:MountingHole_3mm_Pad, F.Cu at (17.8, 167.6)
- added REF**: MountingHole_3mm_Pad, MountingHole:MountingHole_3mm_Pad, F.Cu at (17.8, 20.3)
- moved Cua16 153.9 mm to (251.5, 127.0), turned to 270 degrees
- moved Cua15 145.8 mm to (221.0, 127.0), turned to 270 degrees
- moved Cua14 140.7 mm to (190.5, 127.0), turned to 270 degrees
- moved Cua11 138.0 mm to (99.1, 127.0), turned to 270 degrees
- moved Cub12 132.0 mm to (146.1, 125.7)
- moved Cua13 121.3 mm to (160.0, 127.0), turned to 270 degrees
- moved Rda9 61.0 mm to (34.3, 134.6)
- moved Rdb9 57.3 mm to (34.3, 121.9)
- moved Cua9 53.4 mm to (38.1, 127.0)
- moved Cua12 15.3 mm to (129.5, 127.0), turned to 270 degrees
- moved Rda15 3.59 mm to (217.2, 133.3)
- moved Rda11 3.59 mm to (95.2, 133.3)
- moved Rda12 3.59 mm to (125.7, 133.3)
- moved Rda13 3.59 mm to (156.2, 133.3)
- moved Rda14 3.59 mm to (186.7, 133.3)
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- renumbered Cub17 to Cua11
Routing:
- net VEE: track 649.4 -> 856.4 mm, vias 20 -> 32
- net GND: track 2515.1 -> 2636.2 mm
- net /VO14: track 166.9 -> 188.6 mm
- net Net-(Rda11-Pad1): track 6.35 -> 13.8 mm
- net Net-(Rda16-Pad1): track 6.35 -> 13.8 mm
- net Net-(Rda13-Pad1): track 6.35 -> 13.8 mm
- net Net-(Rda14-Pad1): track 6.35 -> 13.8 mm
- net Net-(Rda15-Pad1): track 6.35 -> 13.8 mm
- net Net-(Rda12-Pad1): track 6.35 -> 13.8 mm
- net /VO12: track 123.9 -> 127.6 mm
- net Net-(Rda11-Pad2): track 7.62 -> 10.2 mm
- net Net-(Rda16-Pad2): track 7.62 -> 10.2 mm
- net Net-(Rda15-Pad2): track 7.62 -> 10.2 mm
- net Net-(Rda14-Pad2): track 7.62 -> 10.2 mm
- net Net-(Rda13-Pad2): track 7.62 -> 10.2 mm
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- added copper zone on B.Cu, net GND

Commit message: Improved the multianem16 board
Moved the power terminal block to the other side of the board.
Parts:
- moved JVIN1 256.9 mm to (273.1, 87.6)
- moved JOUT1 10.9 mm to (21.6, 69.8)
- moved Ra8 3.81 mm to (252.7, 45.7)
- moved Rf8 3.81 mm to (252.7, 76.2)
- moved Rua8 3.81 mm to (252.7, 53.3)
- moved Rb2 3.81 mm to (62.2, 38.1)
- moved Cf10 3.81 mm to (81.3, 118.1)
- moved Cf12 3.81 mm to (142.2, 118.1)
- moved Cf13 3.81 mm to (172.7, 118.1)
- moved Cf14 3.81 mm to (203.2, 118.1)
- moved Cf15 3.81 mm to (233.7, 118.1)
- moved Cf16 3.81 mm to (264.2, 118.1)
- moved Cf3 3.81 mm to (96.5, 69.8)
- moved Cf4 3.81 mm to (127.0, 69.8)
- moved Cf5 3.81 mm to (157.5, 69.8)
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Routing:
- net GND: track 2636.2 -> 2708.1 mm
- net VCC: track 1496.2 -> 1479.7 mm
- net VEE: track 856.4 -> 843.2 mm
- net /VO1: track 43.1 -> 34.5 mm
- net /VO2: track 72.9 -> 65.0 mm
- net /VO3: track 102.6 -> 95.4 mm
- net /VO7: track 224.5 -> 217.4 mm
- net /VO8: track 256.1 -> 248.9 mm
- net /VO6: track 194.1 -> 186.9 mm
- net /VO4: track 132.4 -> 125.9 mm
- net /VO5: track 162.8 -> 156.4 mm

Commit message: Working on new circuit
Changed TerminalBlock footprint to pin header for thermistor probe.
Parts:
- removed REF** (x4): MountingHole_3mm_Pad, MountingHole:MountingHole_3mm_Pad
- added CI1: 100n, Capacitor_THT:C_Rect_L7.2mm_W3.5mm_P5.00mm_FKS2_FKP2_MKS2_MKP2, F.Cu at (35.6, 58.4)
- added CI2: 100n, Capacitor_THT:C_Rect_L7.2mm_W3.5mm_P5.00mm_FKS2_FKP2_MKS2_MKP2, F.Cu at (66.0, 58.4)
- Jw1, Jw10, Jw11, Jw12, Jw13, Jw14, Jw15, Jw16, Jw2, Jw3, Jw4, Jw5, Jw6, Jw7, Jw8, Jw9: footprint TerminalBlock:TerminalBlock_bornier-2_P5.08mm -> Connector_PinHeader_2.54mm:PinHeader_1x02_P2.54mm_Vertical
- moved Cub1 5.24 mm to (36.8, 67.3)
- moved Cub2 5.24 mm to (67.3, 67.3)
- moved Cf1 2.54 mm to (35.6, 72.4), turned to 180 degrees
- moved Cf2 2.54 mm to (66.0, 72.4), turned to 180 degrees
- turned Jw1 to 270 degrees
- turned Jw10 to 90 degrees
- turned Jw11 to 90 degrees
- turned Jw12 to 90 degrees
- turned Jw13 to 90 degrees
- turned Jw14 to 90 degrees
- turned Jw15 to 90 degrees
- turned Jw16 to 90 degrees
- turned Jw2 to 270 degrees
- turned Jw3 to 270 degrees
- turned Jw4 to 270 degrees
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Routing:
- net VCC: track 1479.7 -> 1489.1 mm
- net Net-(CI2-Pad2): track 10.7 -> 18.1 mm
- net Net-(CI1-Pad2): track 10.7 -> 18.1 mm
- net Net-(CI1-Pad1): track 6.66 -> 10.3 mm
- net Net-(CI2-Pad1): track 6.66 -> 10.3 mm
- net Net-(Cf1-Pad1): track 14.1 -> 13.3 mm
- net Net-(Cf2-Pad1): track 14.1 -> 14.8 mm
- removed copper zone on B.Cu, net GND

Commit message: Setting up the the board for the on circuit.
Depending on the offset of the opamp, the circuit will need some help turning on. Getting ready to implement this.
Routing:
- net /VO8: track 248.9 -> 247.8 mm

Commit message: The multianem16 board is almost ready: need to replace Ron by an diode
The problem is that with a resistor every single anemometer is coupled to the others. A diode (1n4148) should isolate them.

The board that I built was kind of poor. Too many flaws in the traces.
Parts:
- added CI10: 100n, Capacitor_THT:C_Rect_L7.2mm_W3.5mm_P5.00mm_FKS2_FKP2_MKS2_MKP2, F.Cu at (81.3, 129.5)
- added CI11: 100n, Capacitor_THT:C_Rect_L7.2mm_W3.5mm_P5.00mm_FKS2_FKP2_MKS2_MKP2, F.Cu at (111.8, 129.5)
- added CI12: 100n, Capacitor_THT:C_Rect_L7.2mm_W3.5mm_P5.00mm_FKS2_FKP2_MKS2_MKP2, F.Cu at (142.2, 129.5)
- added CI13: 100n, Capacitor_THT:C_Rect_L7.2mm_W3.5mm_P5.00mm_FKS2_FKP2_MKS2_MKP2, F.Cu at (172.7, 129.5)
- added CI14: 100n, Capacitor_THT:C_Rect_L7.2mm_W3.5mm_P5.00mm_FKS2_FKP2_MKS2_MKP2, F.Cu at (203.2, 129.5)
- added CI15: 100n, Capacitor_THT:C_Rect_L7.2mm_W3.5mm_P5.00mm_FKS2_FKP2_MKS2_MKP2, F.Cu at (233.7, 129.5)
- added CI16: 100n, Capacitor_THT:C_Rect_L7.2mm_W3.5mm_P5.00mm_FKS2_FKP2_MKS2_MKP2, F.Cu at (264.2, 129.5)
- added CI3: 100n, Capacitor_THT:C_Rect_L7.2mm_W3.5mm_P5.00mm_FKS2_FKP2_MKS2_MKP2, F.Cu at (96.5, 58.5)
- added CI4: 100n, Capacitor_THT:C_Rect_L7.2mm_W3.5mm_P5.00mm_FKS2_FKP2_MKS2_MKP2, F.Cu at (127.0, 58.4)
- added CI5: 100n, Capacitor_THT:C_Rect_L7.2mm_W3.5mm_P5.00mm_FKS2_FKP2_MKS2_MKP2, F.Cu at (157.5, 58.4)
- added CI6: 100n, Capacitor_THT:C_Rect_L7.2mm_W3.5mm_P5.00mm_FKS2_FKP2_MKS2_MKP2, F.Cu at (188.0, 58.4)
- added CI7: 100n, Capacitor_THT:C_Rect_L7.2mm_W3.5mm_P5.00mm_FKS2_FKP2_MKS2_MKP2, F.Cu at (218.4, 58.4)
- added CI8: 100n, Capacitor_THT:C_Rect_L7.2mm_W3.5mm_P5.00mm_FKS2_FKP2_MKS2_MKP2, F.Cu at (248.9, 58.4)
- added CI9: 100n, Capacitor_THT:C_Rect_L7.2mm_W3.5mm_P5.00mm_FKS2_FKP2_MKS2_MKP2, F.Cu at (50.8, 129.5)
- added Coo1: 10u, Capacitor_THT:CP_Radial_D5.0mm_P2.50mm, F.Cu at (276.9, 69.8)
- added D1: 1N4001, Diode_THT:D_DO-41_SOD81_P10.16mm_Horizontal, F.Cu at (254.0, 87.6)
- added Qon1: 2N3906, Package_TO_SOT_THT:TO-92_Inline_Wide, F.Cu at (259.1, 88.9)
- added REF**: MountingHole_3mm_Pad, MountingHole:MountingHole_3mm_Pad, F.Cu at (147.3, 168.9)
- added REF**: MountingHole_3mm_Pad, MountingHole:MountingHole_3mm_Pad, F.Cu at (275.6, 167.6)
- added REF**: MountingHole_3mm_Pad, MountingHole:MountingHole_3mm_Pad, F.Cu at (17.8, 167.6)
- added REF**: MountingHole_3mm_Pad, MountingHole:MountingHole_3mm_Pad, F.Cu at (17.8, 20.3)
- added REF**: MountingHole_3mm_Pad, MountingHole:MountingHole_3mm_Pad, F.Cu at (152.4, 20.3)
- added REF**: MountingHole_3mm_Pad, MountingHole:MountingHole_3mm_Pad, F.Cu at (275.6, 20.3)
- added Ron1: 100, Resistor_THT:R_Axial_DIN0207_L6.3mm_D2.5mm_P15.24mm_Horizontal, F.Cu at (31.8, 39.4)
- added Ron10: 100, Resistor_THT:R_Axial_DIN0207_L6.3mm_D2.5mm_P15.24mm_Horizontal, F.Cu at (85.1, 149.9)
- added Ron11: 100, Resistor_THT:R_Axial_DIN0207_L6.3mm_D2.5mm_P15.24mm_Horizontal, F.Cu at (115.6, 149.9)
- added Ron12: 100, Resistor_THT:R_Axial_DIN0207_L6.3mm_D2.5mm_P15.24mm_Horizontal, F.Cu at (144.8, 146.1)
- added Ron13: 100, Resistor_THT:R_Axial_DIN0207_L6.3mm_D2.5mm_P15.24mm_Horizontal, F.Cu at (176.5, 149.9)
- added Ron14: 100, Resistor_THT:R_Axial_DIN0207_L6.3mm_D2.5mm_P15.24mm_Horizontal, F.Cu at (208.3, 149.9)
- added Ron15: 100, Resistor_THT:R_Axial_DIN0207_L6.3mm_D2.5mm_P15.24mm_Horizontal, F.Cu at (238.8, 149.9)
- added Ron16: 100, Resistor_THT:R_Axial_DIN0207_L6.3mm_D2.5mm_P15.24mm_Horizontal, F.Cu at (269.2, 149.9)
- added Ron2: 100, Resistor_THT:R_Axial_DIN0207_L6.3mm_D2.5mm_P15.24mm_Horizontal, F.Cu at (61.0, 38.1)
- added Ron3: 100, Resistor_THT:R_Axial_DIN0207_L6.3mm_D2.5mm_P15.24mm_Horizontal, F.Cu at (91.4, 38.1)
- added Ron4: 100, Resistor_THT:R_Axial_DIN0207_L6.3mm_D2.5mm_P15.24mm_Horizontal, F.Cu at (120.7, 38.1)
- added Ron5: 100, Resistor_THT:R_Axial_DIN0207_L6.3mm_D2.5mm_P15.24mm_Horizontal, F.Cu at (149.9, 41.9)
- added Ron6: 100, Resistor_THT:R_Axial_DIN0207_L6.3mm_D2.5mm_P15.24mm_Horizontal, F.Cu at (182.9, 38.1)
- added Ron7: 100, Resistor_THT:R_Axial_DIN0207_L6.3mm_D2.5mm_P15.24mm_Horizontal, F.Cu at (214.6, 38.1)
- added Ron8: 100, Resistor_THT:R_Axial_DIN0207_L6.3mm_D2.5mm_P15.24mm_Horizontal, F.Cu at (245.1, 38.1)
- added Ron9: 100, Resistor_THT:R_Axial_DIN0207_L6.3mm_D2.5mm_P15.24mm_Horizontal, F.Cu at (54.6, 149.9)
- added Roo1: 10, Resistor_THT:R_Axial_DIN0207_L6.3mm_D2.5mm_P10.16mm_Horizontal, F.Cu at (266.7, 80.0)
- added Roo2: 22k, Resistor_THT:R_Axial_DIN0207_L6.3mm_D2.5mm_P10.16mm_Horizontal, F.Cu at (276.9, 83.8)
- added Roo3: 4.7k, Resistor_THT:R_Axial_DIN0207_L6.3mm_D2.5mm_P10.16mm_Horizontal, F.Cu at (273.1, 83.8)
- Cua1, Cua10, Cua11, Cua12, Cua13, Cua14, Cua15, Cua16, Cua2, Cua3, Cua4, Cua5, Cua6, Cua7, Cua8, Cua9, Cub1, Cub10, Cub11, Cub12, Cub13, Cub14, Cub15, Cub16, Cub2, Cub3, Cub4, Cub5, Cub6, Cub7, Cub8, Cub9: footprint Capacitor_THT:C_Rect_L7.2mm_W3.5mm_P5.00mm_FKS2_FKP2_MKS2_MKP2 -> Capacitor_THT:C_Disc_D5.0mm_W2.5mm_P2.50mm
- Rb1, Rb10, Rb11, Rb12, Rb13, Rb14, Rb15, Rb16, Rb2, Rb3, Rb4, Rb5, Rb6, Rb7, Rb8, Rb9: footprint Resistor_THT:R_Axial_Power_L20.0mm_W6.4mm_P22.40mm -> Resistor_THT:R_Axial_DIN0414_L11.9mm_D4.5mm_P15.24mm_Horizontal
- moved Cub3 5.08 mm to (96.5, 67.3)
- moved Cub4 5.08 mm to (127.0, 67.3)
- moved Cub5 5.08 mm to (157.4, 67.3)
- moved Cub6 5.08 mm to (188.0, 67.3)
- moved Cub7 5.08 mm to (218.4, 67.3)
- moved Cub8 5.08 mm to (248.9, 67.3)
- moved Cub10 5.08 mm to (81.3, 120.7)
- moved Cub11 5.08 mm to (111.8, 120.7)
- moved Cub12 5.08 mm to (142.2, 120.7)
- moved Cub13 5.08 mm to (172.7, 120.7)
- moved Cub14 5.08 mm to (203.2, 120.7)
- moved Cub15 5.08 mm to (233.7, 120.7)
- moved Cub16 5.08 mm to (264.2, 120.7)
- moved Cub9 5.08 mm to (50.8, 120.7)
- moved Rb2 3.81 mm to (66.0, 38.1)
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Routing:
- net /VON1: track 0.00 -> 1066.9 mm, vias 0 -> 2
- net VCC: track 1489.1 -> 1567.8 mm
- net GND: track 2707.8 -> 2643.2 mm
- net Net-(Coo1-Pad1): track 0.00 -> 18.8 mm
- net Net-(Qon1-Pad2): track 0.00 -> 8.15 mm
- net Net-(CI14-Pad2): track 10.7 -> 18.8 mm
- net Net-(CI3-Pad2): track 10.7 -> 18.1 mm
- net Net-(CI16-Pad2): track 10.7 -> 18.1 mm
- net Net-(CI13-Pad2): track 10.7 -> 18.1 mm
- net Net-(CI15-Pad2): track 10.7 -> 18.1 mm
- net Net-(CI12-Pad2): track 10.7 -> 18.1 mm
- net Net-(CI10-Pad2): track 10.7 -> 18.1 mm
- net Net-(CI11-Pad2): track 10.7 -> 18.1 mm
- net Net-(CI6-Pad2): track 10.7 -> 18.1 mm
- net Net-(Q4-Pad1): track 6.13 -> 12.8 mm
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- added copper zone on B.Cu, net GND

Commit message: Replaced the Ron? resistors by Don? capacitors
I tested the original board and it appeared to be working. Let's try this for real!
Parts:
- removed the REF** at (147.3, 168.9)
- removed the REF** at (152.4, 20.3)
- removed Ron1, Ron10, Ron11, Ron12, Ron13, Ron14, Ron15, Ron16, Ron2, Ron3, Ron4, Ron5, Ron6, Ron7, Ron8, Ron9: 100, Resistor_THT:R_Axial_DIN0207_L6.3mm_D2.5mm_P15.24mm_Horizontal
- added Don1: 1N4148, Diode_THT:D_DO-35_SOD27_P7.62mm_Horizontal, F.Cu at (31.8, 39.4)
- added Don10: 1N4148, Diode_THT:D_DO-35_SOD27_P7.62mm_Horizontal, F.Cu at (85.1, 157.5)
- added Don11: 1N4148, Diode_THT:D_DO-35_SOD27_P7.62mm_Horizontal, F.Cu at (115.6, 157.5)
- added Don12: 1N4148, Diode_THT:D_DO-35_SOD27_P7.62mm_Horizontal, F.Cu at (147.3, 148.6)
- added Don13: 1N4148, Diode_THT:D_DO-35_SOD27_P7.62mm_Horizontal, F.Cu at (176.5, 157.5)
- added Don14: 1N4148, Diode_THT:D_DO-35_SOD27_P7.62mm_Horizontal, F.Cu at (208.3, 157.5)
- added Don15: 1N4148, Diode_THT:D_DO-35_SOD27_P7.62mm_Horizontal, F.Cu at (238.8, 157.5)
- added Don16: 1N4148, Diode_THT:D_DO-35_SOD27_P7.62mm_Horizontal, F.Cu at (269.2, 157.5)
- added Don2: 1N4148, Diode_THT:D_DO-35_SOD27_P7.62mm_Horizontal, F.Cu at (61.0, 30.5)
- added Don3: 1N4148, Diode_THT:D_DO-35_SOD27_P7.62mm_Horizontal, F.Cu at (91.4, 30.5)
- added Don4: 1N4148, Diode_THT:D_DO-35_SOD27_P7.62mm_Horizontal, F.Cu at (120.7, 30.5)
- added Don5: 1N4148, Diode_THT:D_DO-35_SOD27_P7.62mm_Horizontal, F.Cu at (151.8, 36.2)
- added Don6: 1N4148, Diode_THT:D_DO-35_SOD27_P7.62mm_Horizontal, F.Cu at (182.9, 30.5)
- added Don7: 1N4148, Diode_THT:D_DO-35_SOD27_P7.62mm_Horizontal, F.Cu at (214.6, 30.5)
- added Don8: 1N4148, Diode_THT:D_DO-35_SOD27_P7.62mm_Horizontal, F.Cu at (245.1, 30.5)
- added Don9: 1N4148, Diode_THT:D_DO-35_SOD27_P7.62mm_Horizontal, F.Cu at (54.6, 157.5)
- Rua1, Rua10, Rua11, Rua12, Rua13, Rua14, Rua15, Rua16, Rua2, Rua3, Rua4, Rua5, Rua6, Rua7, Rua8, Rua9, Rub1, Rub10, Rub11, Rub12, Rub13, Rub14, Rub15, Rub16, Rub2, Rub3, Rub4, Rub5, Rub6, Rub7, Rub8, Rub9: value 100 -> 10k
Routing:
- net Net-(Don10-Pad1): track 11.7 -> 20.6 mm
- net Net-(Don2-Pad1): track 12.3 -> 20.5 mm
- net Net-(Don9-Pad1): track 11.7 -> 20.0 mm
- net Net-(Don13-Pad1): track 11.7 -> 20.0 mm
- net Net-(Don11-Pad1): track 11.7 -> 20.0 mm
- net Net-(Don7-Pad1): track 11.7 -> 19.4 mm
- net Net-(Don4-Pad1): track 12.8 -> 20.4 mm
- net Net-(Don8-Pad1): track 11.7 -> 19.4 mm
- net Net-(Don3-Pad1): track 12.3 -> 19.9 mm
- net Net-(Don6-Pad1): track 12.3 -> 19.9 mm
- net Net-(Don16-Pad1): track 12.3 -> 19.9 mm
- net Net-(Don14-Pad1): track 12.3 -> 19.9 mm
- net Net-(Don15-Pad1): track 12.3 -> 19.9 mm
- net /VON1: track 1066.9 -> 1074.5 mm, vias 2 -> 3
- net GND: track 2643.2 -> 2639.4 mm
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